File: electrical/uc_module.kicad_sch (KiCad schematic)
At the start: 12 parts, among them J6 Conn_01x06_Pin, SW2 SW_SPST, U1 ATtiny84A-PU

Commit message: Względenie działa
Parts:
- removed J6: Conn_01x06_Pin, symbol Connector:Conn_01x05_Pin
- added C10, C2: 15n, symbol Device:C
- added D3, D9: 1N4148, Diode_THT:D_DO-35_SOD27_P7.62mm_Horizontal, symbol Diode:1N4148
- added J6: Conn_01x06_Pin, symbol Connector:Conn_01x06_Pin
- added J7: Conn_01x01_Pin, symbol Connector:Conn_01x01_Pin
- added J8, J9: Screw_Terminal_01x01, symbol Connector:Screw_Terminal_01x01
- added R13: 1k, symbol Device:R
- added SW3: NEUTRAL DETECT, symbol Switch:SW_SPST
- added SW4: OLI PRESSURE SWITCH, symbol Switch:SW_SPST
- R11: value 1k -> 3.3k
- R8: value 470 -> 1k
- R9: value 12k -> 15k
Connections:
- net +5V: now also R13.2
- net GND: now also C10.2, C2.2, SW3.1 (A), SW4.1 (A)
- net NEUTRAL: now also C10.1, D9.2 (A)
- net OLI PRESSURE: now also C2.1, D3.2 (A), R13.1
- new net GND when NO oli pressure: D3.1 (K), J8.1 (Pin_1), SW4.2 (B)
- new net GND when no gear engaged: D9.1 (K), J9.1 (Pin_1), SW3.2 (B)
Other:
- note removed: "Depending on LED used"
- moved on the sheet: D6, R11, R8, R9
